Commit message: go2 model update

File: LidarSim2Real/go2_urdf_modified/urdf/go2_description.urdf (robot description, URDF)
Before this commit: robot go2_description, 33 links, 32 joints
Links:
- link FL_calf: geometry collision cylinder length=0.12 radius=0.012; visual mesh filename=dae/calf.dae
- link FL_foot: geometry collision sphere radius=0.022; visual mesh filename=dae/foot.dae
- link FL_hip: geometry collision cylinder length=0.04 radius=0.046; visual mesh filename=dae/hip.dae
- link FL_thigh: geometry collision box size=0.213 0.0245 0.034; visual mesh filename=dae/thigh.dae
- link FR_calf: geometry collision cylinder length=0.12 radius=0.013; visual mesh filename=dae/calf_mirror.dae
- link FR_foot: geometry collision sphere radius=0.022; visual mesh filename=dae/foot.dae
- link FR_hip: geometry collision cylinder length=0.04 radius=0.046; visual mesh filename=dae/hip.dae
- link FR_thigh: geometry collision box size=0.213 0.0245 0.034; visual mesh filename=dae/thigh_mirror.dae
- link RL_calf: geometry collision cylinder length=0.12 radius=0.013; visual mesh filename=dae/calf.dae
- link RL_foot: geometry collision sphere radius=0.022; visual mesh filename=dae/foot.dae
- link RL_hip: geometry collision cylinder length=0.04 radius=0.046; visual mesh filename=dae/hip.dae
- link RL_thigh: geometry collision box size=0.213 0.0245 0.034; visual mesh filename=dae/thigh.dae
- link RR_calf: geometry collision cylinder length=0.12 radius=0.013; visual mesh filename=dae/calf_mirror.dae
- link RR_foot: geometry collision sphere radius=0.022; visual mesh filename=dae/foot.dae
- link RR_hip: geometry collision cylinder length=0.04 radius=0.046; visual mesh filename=dae/hip.dae
- link RR_thigh: geometry collision box size=0.213 0.0245 0.034; visual mesh filename=dae/thigh_mirror.dae
- link base: geometry collision box size=0.3762 0.0935 0.114; visual mesh filename=dae/base.dae
- link jetson_box_link: geometry collision box size=0.185 0.105 0.03; visual mesh filename=dae/jetson_box.dae
- link mid360withcase_link: geometry collision mesh filename=dae/mid360withcase.stl scale=0.001 0.001 0.001; visual mesh filename=dae/mid360withcase.stl scale=0.001 0.001 0.001

Commit message: go2 description change

File: LidarSim2Real/go2_urdf_modified/urdf/go2_description.urdf (robot description, URDF)
Before this commit: robot go2_description, 33 links, 32 joints
Links:
- link mid360withcase_link: geometry collision mesh filename=dae/mid360withcase.dae scale=1 1 1; visual mesh filename=dae/mid360withcase.dae scale=1 1 1
